File: Hardware/AQS.sch (EAGLE design)
At the start: 43 parts, among them IC1 BME680, IC2 CP2102N-A01-GQFN24, IC4 ESPWROOM32, J1 ESP-PROG-2X3-1.27-SHROUDED, J2 M02X5-1.27-S, J3 USB-C-16P-16P, Q1 MMDT3904, Q2 2N7002

Commit message: Finished major rework for v3.0 release
Parts:
- removed IC4: ESPWROOM32, SuperHouse-MCUs:ESPWROOM32
- added IC3: BME680, SuperHouse-Sensors:BME680
- added U$23, U$24, U$25: FIDUCIAL1X2, SuperHouse-Symbols:FIDUCIAL1X2
- C2, C3: device SuperHouse-DiscreteSemi:CAP0603 -> SuperHouse-DiscreteSemi:CAP0805
- C5: value 10uF 50V -> 10uF
- IC1: value BME680 -> ESPWROOM32; device SuperHouse-Sensors:BME680 -> SuperHouse-MCUs:ESPWROOM32
- LED2: value WS2812B5050 -> TX/YEL; device SuperHouse-LEDs:WS2812B5050 -> SuperHouse-LEDs:LED0603
- LED5: value TX/YEL -> WS2812B5050; device SuperHouse-LEDs:LED0603 -> SuperHouse-LEDs:WS2812B5050
- R1: value 10K -> 1K
- R10: value 5.1K -> 10K
- R11: value 22K -> 10K
- R13: value 4K7 -> 22K
- R14: value 4K7 -> 22.1K
- R15: value 4K7 -> 47.5K
- R2: value 22.1K -> 1K
- R3: value 47.5K -> 4K7
- R5: value 10K -> 4K7
- R6: value 5.1K -> 4K7
- R7: value 10K -> 5.1K
- R8: value 1K -> 5.1K
- R9: value 1K -> 10K
- renumbered C12 to C7, LED6 to LED3
Connections:
- removed net GPIO13: IC4.IO13, Q2.S, R4.1
- removed net GPIO2: IC4.IO2, LCD.DC
- removed net GPIO23: IC4.IO23
- removed net GPIO4: IC4.IO4
- removed net TFT_CIPO: IC4.IO19
- removed net TFT_CS: IC4.IO26
- removed net TFT_RESET: LCD.RES
- new net TFT_DC: IC1.IO2, LCD.DC
- new net TFT_RST: IC1.IO4, LCD.!RST
- new net WS2812B: IC1.IO13, Q2.S, R4.1
- net !RESET: now also IC1.EN, R13.2; no longer IC4.EN, R11.2
- net 3.3V: now also IC1.3V3, IC3.CSB, IC3.VDD, IC3.VDDIO, LED2.A, R13.1, R5.2, R6.2, R9.2; no longer IC1.CSB, IC1.VDD, IC1.VDDIO, IC4.3V3, LED5.A, R1.2, R11.1, R14.2, R15.2
- net 5V: now also LED5.VDD, R14.2, R3.2; no longer LED2.VDD, R13.2, R2.2
- net DTR: now also R10.1; no longer R5.1
- net GND: now also IC1.GND@1, IC1.GND@2, IC1.GND@3, IC1.GND@4, IC3.GND, IC3.SDO, LED5.GND, R15.1, R7.1, R8.1; no longer IC1.GND, IC1.SDO, IC4.GND@1, IC4.GND@2, IC4.GND@3, IC4.GND@4, LED2.GND, R10.1, R3.1, R6.1
- net GPIO0: now also IC1.IO0; no longer IC4.IO0
- net H1: now also LED4.DI, R3.1; no longer LED2.DI, R13.1
- net N$1: now also R9.1; no longer R1.1
- net N$10: now also R8.2; no longer R10.2
- net N$11: now also R7.2; no longer R6.2
- net N$12: now also LED4.DO, LED5.DI; no longer LED2.DO, LED4.DI
- net N$13: now also LED2.C, R1.2; no longer LED5.C, R9.2
- net N$2: now also R2.2; no longer R8.2
- net N$39: now also R14.1, R15.2; no longer R2.1, R3.2
- net N$7: now also R10.2; no longer R5.2
- net N$8: now also R11.2; no longer R7.2
- net PMS_RESET: now also IC1.IO27; no longer IC4.IO27
- net PMS_RX: now also IC1.IO17; no longer IC4.IO17
- net PMS_SET: now also IC1.IO25; no longer IC4.IO25
- net PMS_TX: now also IC1.IO16; no longer IC4.IO16
- net RTS: now also R11.1; no longer R7.1
- net RXD0: now also IC1.RXD0; no longer IC4.RXD0
- net RX_LED: now also R2.1; no longer R8.1
- net SCL: now also IC1.IO22, IC3.SCK, R6.1; no longer IC1.SCK, IC4.IO22, R14.1
- net SDA: now also IC1.IO21, IC3.SDI, R5.1; no longer IC1.SDI, IC4.IO21, R15.1
- net TFT_COPI: now also IC1.IO23, LCD.COPI; no longer LCD.SDA
- net TFT_SCLK: now also IC1.IO18, LCD.SCLK; no longer IC4.IO18, LCD.SCK
- net TXD0: now also IC1.TXD0; no longer IC4.TXD0
- net TX_LED: now also R1.1; no longer R9.1
Other:
- note added: "GPIO0: Button (active low) GPIO1: USB_TX GPIO2: TFT_DC GPIO3: USB_RX GPIO4: TFT_RST GPIO13: WS2812B GPIO16: PMS_TX (RX2 of MCU) GPIO17: PMS_RX (TX2 of MCU) GPIO18: TFT_SCLK GPIO21: SDA GPIO22: SCL GPIO23: TFT_COPI GPIO25: PMS_SET GPIO27: PMS_RESET Firmware: https://github.com/openairproject/sensor-esp32"
- note added: "I2C Addresses: 0x77: BME680"
- note removed: "GPIO0: Button (active low) GPIO1: USB_TX GPIO2: TFT_DC GPIO3: USB_RX GPIO4: TFT_RST GPIO13: WS2812B GPIO16: PMS_TX (RX2 of MCU) GPIO17: PMS_RX (TX2 of MCU) GPIO18: TFT_SCLK GPIO19: TFT_MISO GPIO21: SDA GPIO22: SCL GPIO23: TFT_MOSI GPIO25: PMS_SET GPIO26: TFT_CS GPIO27: PMS_RESET Firmware: https://github.com/openairproject/sensor-esp32"
- note removed: "I2C Address: 0x77: BME680"
- moved on the sheet: R1, R10, R11, R2, R7, R8, R9

Commit message: Major restructure to reduce size of PCB. ERC and DRC for v3.0 release.
Parts:
- removed C6, C8: 100nF, SuperHouse-DiscreteSemi:CAP0603
- removed J3: USB-C-16P-16P, SuperHouse-Connectors:USB-C-16P-16P
- removed LCD: OLED-SPI-HEADER, SuperHouse-Displays:OLED-SPI-HEADER
- removed LED4, LED5: WS2812B5050, SuperHouse-LEDs:WS2812B5050
- removed Q2: 2N7002, SuperHouse-DiscreteSemi:MOSFET-NCHANNEL-233
- removed R3, R4: 4K7, SuperHouse-DiscreteSemi:RESISTOR0603
- removed R7, R8: 5.1K, SuperHouse-DiscreteSemi:RESISTOR0603
- added MOD1: OLED-SPI-CS-PINS, SuperHouse-Displays:OLED-SPI-CS-PINS
- F1: device SuperHouse-Fuses:PTC050 -> SuperHouse-Fuses:PTC-1206
- J1: value ESP-PROG-2X3-1.27-SHROUDED -> USB; device SuperHouse-ESP-Prog:ESP-PROG-2X3-1.27-SHROUDED -> SuperHouse-Connectors:USB-B-5P-VERT
- S2: device SuperHouse-Switches:TAC_SWITCH_2PINSMT -> SuperHouse-Switches:TAC_SWITCH-PTH-4.5
Connections:
- net PMS_RESET renamed IO27_PMS_RESET
- net PMS_RX renamed IO17_PMS_RX
- net PMS_SET renamed IO25_PMS_SET
- net PMS_TX renamed IO16_PMS_TX
- net SCL renamed IO22_SCL
- net SDA renamed IO21_SDA
- removed net H1: LED4.DI, Q2.D, R3.1
- removed net N$10: J3.CC2, R8.2
- removed net N$11: J3.CC1, R7.2
- removed net N$12: LED4.DO, LED5.DI
- removed net TFT_COPI: IC1.IO23, LCD.COPI
- removed net TFT_DC: IC1.IO2, LCD.DC
- removed net TFT_RST: IC1.IO4, LCD.!RST
- removed net TFT_SCLK: IC1.IO18, LCD.SCLK
- removed net VIN: F1.1, J3.VBUS
- removed net WS2812B: IC1.IO13, Q2.S, R4.1
- new net IO13: IC1.IO13
- new net IO14_TFT_BLK: IC1.IO14, MOD1.BLK
- new net IO18_SCLK: IC1.IO18, MOD1.SCK
- new net IO23_COPI: IC1.IO23, MOD1.COPI
- new net IO26_TFT_CS: IC1.IO26, MOD1.!CS
- new net IO2_TFT_DC: IC1.IO2, MOD1.DC
- new net IO4_TFT_RST: IC1.IO4, MOD1.!RST
- new net N$3: F1.1, J1.VBUS
- net !RESET: now also S2.3, S2.4; no longer J1.CH_EN, S2.S
- net 3.3V: now also MOD1.VCC; no longer J1.VDD, LCD.VCC, Q2.G, R4.2
- net 5V: no longer C6.1, C8.1, LED4.VDD, LED5.VDD, R3.2
- net D+: now also J1.D+; no longer J3.D+
- net D-: now also J1.D-; no longer J3.D-
- net GND: now also MOD1.GND, S2.1, S2.2; no longer C6.2, C8.2, J3.GND, LCD.GND, LED4.GND, LED5.GND, R7.1, R8.1, S2.P
- net GPIO0: no longer J1.GPIO0
- net RXD0: no longer J1.ESP_RX
- net TXD0: no longer J1.ESP_TX
Other:
- note added: "(C)2021 SuperHouse Automation: www.superhouse.tv"
- note added: "IO0: Button (active low) IO1: USB_TX IO2: TFT_DC IO3: USB_RX IO4: TFT_RST IO13: WS2812B IO16: PMS_TX (RX2 of MCU) IO17: PMS_RX (TX2 of MCU) IO18: SCLK IO21: SDA IO22: SCL IO23: COPI IO25: PMS_SET IO26: TFT_CS IO27: PMS_RESET Firmware: https://github.com/openairproject/sensor-esp32"
- note added: "Licensed under the TAPR Open Hardware License: www.tapr.org/ohl"
- note added: "To Do: put WS2812B back on?"
- note added: "V3.0 (2021-09-16)"
- note removed: "ESP-Prog Header"
- note removed: "GPIO0: Button (active low) GPIO1: USB_TX GPIO2: TFT_DC GPIO3: USB_RX GPIO4: TFT_RST GPIO13: WS2812B GPIO16: PMS_TX (RX2 of MCU) GPIO17: PMS_RX (TX2 of MCU) GPIO18: TFT_SCLK GPIO21: SDA GPIO22: SCL GPIO23: TFT_COPI GPIO25: PMS_SET GPIO27: PMS_RESET Firmware: https://github.com/openairproject/sensor-esp32"
- note removed: "RGB LEDs"
- note removed: "USB-C Connection"
- note removed: "V3.0 (2020-07-16)"
- moved on the sheet: C1, C2, C3, C7, F1, IC2, IC3, LED1, LED2, LED3, R1, R14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
